Commit message: correct placement of imu

File: src/felix_description/urdf/felix.urdf.xacro (robot description, xacro)
@@ -4,4 +4,5 @@
   TF tree:  base_footprint -> base_link -> imu_link
                                         -> laser
+                                        -> camera_link
   base_link sits at the chassis rotation centre (the point the EKF publishes
   odom -> base_link for); base_footprint is its ground projection. robot_state_
@@ -34,9 +35,10 @@
   <xacro:property name="laser_z"   value="0.0665"/>
   <xacro:property name="laser_yaw" value="3.14159265"/>
-  <!-- IMU mount, base_link -> imu_link.  Identity for now: the EKF only fuses
-       gyro yaw-rate, which is invariant to rotation about the shared z-axis, so
-       this does not affect localisation. The board's in-plane accel axes are
-       left-handed vs the robot (IMU +y ~ forward, +x ~ left); only encode the
-       real roll/pitch/yaw here if/when you start fusing acceleration. -->
+  <!-- IMU mount, base_link -> imu_link.  Identity: the EKF only fuses gyro
+       yaw-rate, which is invariant to rotation about the shared z-axis, so this
+       does not affect localisation. IMU re-mounted x-forward + centered (2026-06).
+       The raw gyro-Z is board-intrinsically inverted vs REP-103 and is corrected
+       in bridge_node._publish_imu (not here). Accel is published raw and unfused;
+       encode real roll/pitch/yaw here only if/when you start fusing acceleration. -->
   <xacro:property name="imu_x"     value="0.0"/>
   <xacro:property name="imu_y"     value="0.0"/>
@@ -45,4 +47,19 @@
   <xacro:property name="imu_pitch" value="0.0"/>
   <xacro:property name="imu_yaw"   value="0.0"/>
+  <!-- CAMERA mount, base_link -> camera_link.  Measured 2026-06-08:
+       horizontally centred (y=0). z=0: the camera centre is wheel_radius
+       (0.0485 m) above the ground, which is exactly base_link's height (axle
+       height), so the offset relative to base_link is zero.
+       x: the camera base sits ~10 mm behind the front-most point of the front
+       wheels. Front axle = wheel_base/2 = 0.095 m forward; front-most wheel point
+       = 0.095 + wheel_radius (0.0485) = 0.1435 m; minus 0.010 = 0.1335 m.
+       Orientation is REP-103 (x forward) like base_link; the REP-105 optical
+       frame (z forward) gets added when felix_perception lands. -->
+  <xacro:property name="camera_x"     value="0.1335"/>
+  <xacro:property name="camera_y"     value="0.0"/>
+  <xacro:property name="camera_z"     value="0.0"/>
+  <xacro:property name="camera_roll"  value="0.0"/>
+  <xacro:property name="camera_pitch" value="0.0"/>
+  <xacro:property name="camera_yaw"   value="0.0"/>
   <!-- ===================== Materials ===================== -->
   <material name="felix_grey"><color rgba="0.25 0.27 0.30 1.0"/></material>
@@ -82,3 +99,16 @@
     <origin xyz="${laser_x} ${laser_y} ${laser_z}" rpy="0 0 ${laser_yaw}"/>
   </joint>
+  <link name="camera_link">
+    <visual>
+      <origin xyz="0 0 0" rpy="0 0 0"/>
+      <geometry><box size="0.025 0.09 0.025"/></geometry>
+      <material name="felix_black"/>
+    </visual>
+  </link>
+  <joint name="base_link_to_camera" type="fixed">
+    <parent link="base_link"/>
+    <child link="camera_link"/>
+    <origin xyz="${camera_x} ${camera_y} ${camera_z}"
+            rpy="${camera_roll} ${camera_pitch} ${camera_yaw}"/>
+  </joint>
 </robot>

Commit message: added localization

File: src/felix_description/urdf/felix.urdf.xacro (robot description, xacro)
@@ -25,14 +25,16 @@
        0-degree ray relative to robot forward (+x). If the scan appears rotated
        in rviz/the map, adjust laser_yaw (RPLIDAR zero often faces the cable). -->
-  <!-- Measured 2026-06-07: 0.08 m forward, centred, beam 0.115 m above floor.
-       laser_z is relative to base_link (axle height), = 0.115 - wheel_radius.
-       laser_yaw = pi: the RPLIDAR is mounted rotated 180deg (zero-ray faces
-       backward). Verified live: a wall squarely ~1m in FRONT of the robot
-       appeared at lidar bearing ~180deg; without this the map drifted badly
-       (scans fought the odometry, robot appeared to drive through walls). -->
-  <xacro:property name="laser_x"   value="0.08"/>
+  <!-- laser_x measured 2026-06-08: 2.5 in = 0.0635 m, the forward distance from
+       base_link's origin (chassis rotation centre) to the lidar's scan-centre axis.
+       centred (laser_y = 0); beam 0.115 m above floor, so laser_z = 0.115 -
+       wheel_radius relative to base_link (axle height).
+       laser_yaw = 0: the RPLIDAR was physically re-oriented 2026-06-08 so its
+       zero-ray faces FORWARD (+x), so no yaw correction is needed. (Previously it
+       was mounted rotated 180deg with the zero-ray facing backward, which needed
+       laser_yaw = pi.) -->
+  <xacro:property name="laser_x"   value="0.0635"/>
   <xacro:property name="laser_y"   value="0.0"/>
   <xacro:property name="laser_z"   value="0.0665"/>
-  <xacro:property name="laser_yaw" value="3.14159265"/>
+  <xacro:property name="laser_yaw" value="0.0"/>
   <!-- IMU mount, base_link -> imu_link.  Identity: the EKF only fuses gyro
        yaw-rate, which is invariant to rotation about the shared z-axis, so this

Commit message: add navigation

File: src/felix_description/urdf/felix.urdf.xacro (robot description, xacro)
@@ -2,12 +2,14 @@
 <!--
   Felix mecanum chassis description.
-  TF tree:  base_footprint -> base_link -> imu_link
-                                        -> laser
-                                        -> camera_link
-  base_link sits at the chassis rotation centre (the point the EKF publishes
-  odom -> base_link for); base_footprint is its ground projection. robot_state_
-  publisher turns the fixed joints below into /tf_static, which is what the EKF
-  (base_link -> imu_link) and SLAM (base_link -> laser) consume; this replaces
-  the temporary static_transform_publisher that bringup used before.
+  TF tree:  base_link -> base_footprint   (ground projection, below)
+                      -> imu_link
+                      -> laser
+                      -> camera_link
+  base_link is the URDF ROOT and the chassis rotation centre (the point the EKF
+  publishes odom -> base_link for). Everything else, including base_footprint (the
+  ground projection), hangs off it, so base_link has exactly one parent (odom),
+  not two. robot_state_publisher turns the fixed joints below into /tf_static, which
+  is what the EKF (base_link -> imu_link) and SLAM (base_link -> laser) consume; this
+  replaces the temporary static_transform_publisher that bringup used before.
   >>> EDIT THE MOUNT OFFSETS BELOW TO YOUR MEASURED VALUES <<<
   All offsets are in metres / radians, in REP-103 base_link axes:
@@ -77,9 +79,14 @@
     </visual>
   </link>
-  <joint name="base_footprint_to_base_link" type="fixed">
-    <parent link="base_footprint"/>
-    <child link="base_link"/>
-    <!-- Lift base_link to axle height above the ground projection. -->
-    <origin xyz="0 0 ${wheel_radius}" rpy="0 0 0"/>
+  <!-- base_footprint is a CHILD of base_link, not its parent: the EKF publishes
+       odom -> base_link, so base_link is the tree node odom drives. If base_footprint
+       parented base_link here, base_link would have two parents (odom + base_footprint),
+       an illegal TF tree that places the body and the sensors via different paths
+       (body mirrors/drifts away from the laser). base_footprint is the ground
+       projection, so it sits wheel_radius BELOW base_link. -->
+  <joint name="base_link_to_base_footprint" type="fixed">
+    <parent link="base_link"/>
+    <child link="base_footprint"/>
+    <origin xyz="0 0 ${-wheel_radius}" rpy="0 0 0"/>
   </joint>
   <link name="imu_link"/>

Commit message: perception with yolo

File: src/felix_description/urdf/felix.urdf.xacro (robot description, xacro)
@@ -5,5 +5,5 @@
                       -> imu_link
                       -> laser
-                      -> camera_link
+                      -> camera_link -> camera_optical_link  (REP-105 optical, z fwd)
   base_link is the URDF ROOT and the chassis rotation centre (the point the EKF
   publishes odom -> base_link for). Everything else, including base_footprint (the
@@ -59,5 +59,7 @@
        = 0.095 + wheel_radius (0.0485) = 0.1435 m; minus 0.010 = 0.1335 m.
        Orientation is REP-103 (x forward) like base_link; the REP-105 optical
-       frame (z forward) gets added when felix_perception lands. -->
+       frame (z forward, x right, y down) is published as camera_optical_link,
+       a fixed child of camera_link (below). felix_perception stamps CameraInfo
+       and Detection2DArray in camera_optical_link, not camera_link. -->
   <xacro:property name="camera_x"     value="0.1335"/>
   <xacro:property name="camera_y"     value="0.0"/>
@@ -121,3 +123,13 @@
             rpy="${camera_roll} ${camera_pitch} ${camera_yaw}"/>
   </joint>
+  <!-- REP-105 optical frame: z forward, x right, y down. Standard REP-103
+       (x forward) -> optical rotation is rpy = (-pi/2, 0, -pi/2). felix_perception
+       back-projects pixels and stamps detections/CameraInfo in this frame; the
+       fusion node transforms the bearing wedge camera_optical_link -> laser. -->
+  <link name="camera_optical_link"/>
+  <joint name="camera_to_camera_optical" type="fixed">
+    <parent link="camera_link"/>
+    <child link="camera_optical_link"/>
+    <origin xyz="0 0 0" rpy="${-pi/2} 0 ${-pi/2}"/>
+  </joint>
 </robot>

Commit message: support for nemotron

File: src/felix_description/urdf/felix.urdf.xacro (robot description, xacro)
@@ -27,16 +27,17 @@
        0-degree ray relative to robot forward (+x). If the scan appears rotated
        in rviz/the map, adjust laser_yaw (RPLIDAR zero often faces the cable). -->
-  <!-- laser_x measured 2026-06-08: 2.5 in = 0.0635 m, the forward distance from
-       base_link's origin (chassis rotation centre) to the lidar's scan-centre axis.
-       centred (laser_y = 0); beam 0.115 m above floor, so laser_z = 0.115 -
-       wheel_radius relative to base_link (axle height).
-       laser_yaw = 0: the RPLIDAR was physically re-oriented 2026-06-08 so its
-       zero-ray faces FORWARD (+x), so no yaw correction is needed. (Previously it
-       was mounted rotated 180deg with the zero-ray facing backward, which needed
-       laser_yaw = pi.) -->
-  <xacro:property name="laser_x"   value="0.0635"/>
+  <!-- laser_x/z measured 2026-06-21 for the RPLIDAR A2 M12 re-mount: 0.083 m
+       forward and 0.075 m up from base_link's origin (the chassis rotation centre,
+       at axle height), centred (laser_y = 0). Both offsets are relative to
+       base_link directly, NOT the floor (do not subtract wheel_radius).
+       laser_yaw = pi: the A2 M12 is mounted with its zero-degree ray facing
+       BACKWARD (the cable side faces the rear), so the scan is rotated 180deg:
+       a target behind the robot shows up in front without this correction. (The
+       PREVIOUS unit was physically turned to face forward on 2026-06-08 and used
+       laser_yaw = 0; this new unit went back to the rear-facing orientation.) -->
+  <xacro:property name="laser_x"   value="0.083"/>
   <xacro:property name="laser_y"   value="0.0"/>
-  <xacro:property name="laser_z"   value="0.0665"/>
-  <xacro:property name="laser_yaw" value="0.0"/>
+  <xacro:property name="laser_z"   value="0.075"/>
+  <xacro:property name="laser_yaw" value="${pi}"/>
   <!-- IMU mount, base_link -> imu_link.  Identity: the EKF only fuses gyro
        yaw-rate, which is invariant to rotation about the shared z-axis, so this
